File: 2024-Electrical-Vanguard_V2/Vanguard/Vanguard_V2/Vanguard_new.kicad_sch (KiCad schematic)
At the start: 72 parts, among them J1 USB_C, J2 Conn_02x03_Pin, J3 Micro_SD_Card_Det1, J4 STARBOARD_SERVO, J5 PORTSIDE_SERVO, J6 Conn_01x02_Pin, Q1 BSS138, Q2 BSS138, Q3 BSS138, Q4 BSS138, U1 ATSAMD11D14A-M, U2 ATmega4809-A, U3 AT25DF641A-SH-T, U4 AP2112K-3.3, U5 MPM3610AGQV-P, U6 BNO086, U7 TXB0104D, U8 TPS61092, Y1 32.768kHz

Commit message: some changes in the schematic
Connections:
- net GND: no longer D6.1 (K)
- net VCC: no longer U5.2 (VCC)
- net at C5.1, R15.1, U4.1 (VIN)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: now also D6.1 (K)
Other:
- moved on the sheet: D6
Changed lines of the file:
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@@
 	)
 	(junction
-		(at 288.29 58.42)
-		(diameter 0)
-		(color 0 0 0 0)
-	)
-	(junction
 		(at 96.52 26.67)
 		(diameter 0)
@@
 	(wire
 		(pts
+			(xy 340.36 25.4) (xy 341.63 25.4)
+		)
+		(stroke
+			(width 0)
+			(type default)
+		)
+	)
+	(wire
+		(pts
 			(xy 304.8 119.38) (xy 311.15 119.38)
 		)
@@
 	(wire
 		(pts
+			(xy 341.63 25.4) (xy 341.63 44.45)
+		)
+		(stroke
+			(width 0)
+			(type default)
+		)
+	)
+	(wire
+		(pts
 			(xy 109.22 58.42) (xy 118.11 58.42)
 		)
@@
 	(wire
 		(pts
-			(xy 288.29 58.42) (xy 290.83 58.42)
-		)
-		(stroke
-			(width 0)
-			(type default)
-		)
-	)
-	(wire
-		(pts
 			(xy 67.31 20.32) (xy 66.04 20.32)
 		)
@@
 	(wire
 		(pts
-			(xy 283.21 58.42) (xy 288.29 58.42)
-		)
-		(stroke
-			(width 0)
-			(type default)
-		)
-	)
-	(wire
-		(pts
 			(xy 256.54 57.15) (xy 256.54 60.96)
 		)
@@
 	(wire
 		(pts
+			(xy 325.12 25.4) (xy 332.74 25.4)
+		)
+		(stroke
+			(width 0)
+			(type default)
+		)
+	)
+	(wire
+		(pts
 			(xy 339.09 170.18) (xy 344.17 170.18)
 		)
@@
 	(text "INPUT USB"
 		(exclude_from_sim no)
-		(at 244.094 22.352 0)
+		(at 192.278 17.526 0)
 		(effects
 			(font
@@
 	(text "POWER STABILIZATION"
 		(exclude_from_sim no)
-		(at 301.244 22.352 0)
+		(at 299.72 18.796 0)
 		(effects
 			(font
@@
 		)
 	)
-	(global_label "VBUS_out"
-		(shape input)
-		(at 283.21 58.42 180)
-		(fields_autoplaced yes)
-		(effects
-			(font
-				(size 1.27 1.27)
-			)
-			(justify right)
-		)
-		(property "Intersheetrefs" "${INTERSHEET_REFS}"
-			(at 271.3349 58.42 0)
-			(effects
-				(font
-					(size 1.27 1.27)
-				)
-				(justify right)
-				(hide yes)
-			)
-		)
-	)
 	(global_label "RST"
 		(shape input)
@@
 	(global_label "VBUS_out"
 		(shape input)
-		(at 331.47 30.48 180)
+		(at 325.12 25.4 180)
 		(fields_autoplaced yes)
 		(effects
@@
 		)
 		(property "Intersheetrefs" "${INTERSHEET_REFS}"
-			(at 319.5949 30.48 0)
+			(at 313.2449 25.4 0)
 			(effects
 				(font
@@
 	)
 	(symbol
-		(lib_id "power:VCC")
-		(at 288.29 58.42 180)
-		(unit 1)
-		(exclude_from_sim no)
-		(in_bom yes)
-		(on_board yes)
-		(dnp no)
-		(property "Reference" "#PWR068"
-			(at 288.29 54.61 0)
-			(effects
-				(font
-					(size 1.27 1.27)
-				)
-				(hide yes)
-			)
-		)
-		(property "Value" "VCC"
-			(at 289.56 63.246 0)
-			(effects
-				(font
-					(size 1.27 1.27)
-				)
-			)
-		)
-		(property "Footprint" ""
-			(at 288.29 58.42 0)
-			(effects
-				(font
-					(size 1.27 1.27)
-				)
-				(hide yes)
-			)
-		)
-		(property "Datasheet" ""
-			(at 288.29 58.42 0)
-			(effects
-				(font
-					(size 1.27 1.27)
-				)
-				(hide yes)
-			)
-		)
-		(property "Description" "Power symbol creates a global label with name \"VCC\""
-			(at 288.29 58.42 0)
-			(effects
-				(font
-					(size 1.27 1.27)
-				)
-				(hide yes)
-			)
-		)
-		(pin "1"
-		)
-		(instances
-			(project "Vanguard_new"
-				(path "/972fbf12-2dcd-4fdf-b1c9-8a2880c46640"
-					(reference "#PWR068")
-					(unit 1)
-				)
-			)
-		)
-	)
-	(symbol
 		(lib_id "power:+3.3V")
 		(at 248.92 49.53 0)
@@
 	)
 	(symbol
-		(lib_id "power:GND")
-		(at 339.09 30.48 90)
-		(unit 1)
-		(exclude_from_sim no)
-		(in_bom yes)
-		(on_board yes)
-		(dnp no)
-		(fields_autoplaced yes)
-		(property "Reference" "#PWR034"
-			(at 345.44 30.48 0)
-			(effects
-				(font
-					(size 1.27 1.27)
-				)
-				(hide yes)
-			)
-		)
-		(property "Value" "GND"
-			(at 342.9 30.4799 90)
-			(effects
-				(font
-					(size 1.27 1.27)
-				)
-				(justify right)
-			)
-		)
-		(property "Footprint" ""
-			(at 339.09 30.48 0)
-			(effects
-				(font
-					(size 1.27 1.27)
-				)
-				(hide yes)
-			)
-		)
-		(property "Datasheet" ""
-			(at 339.09 30.48 0)
-			(effects
-				(font
-					(size 1.27 1.27)
-				)
-				(hide yes)
-			)
-		)
-		(property "Description" "Power symbol creates a global label with name \"GND\" , ground"
-			(at 339.09 30.48 0)
-			(effects
-				(font
-					(size 1.27 1.27)
-				)
-				(hide yes)
-			)
-		)
-		(pin "1"
-		)
-		(instances
-			(project "Vanguard_new"
-				(path "/972fbf12-2dcd-4fdf-b1c9-8a2880c46640"
-					(reference "#PWR034")
-					(unit 1)
-				)
-			)
-		)
-	)
-	(symbol
 		(lib_id "AT25DF641A-SH-T:AT25DF641A-SH-T")
 		(at 170.18 233.68 0)
@@
 	(symbol
 		(lib_id "Diode:PMEG6020ER")
-		(at 335.28 30.48 180)
+		(at 336.55 25.4 180)
 		(unit 1)
 		(exclude_from_sim no)
@@
 		(fields_autoplaced yes)
 		(property "Reference" "D6"
-			(at 335.5975 24.13 0)
+			(at 336.8675 19.05 0)
 			(effects
 				(font
@@
 		)
 		(property "Value" "PMEG6020ER"
-			(at 335.5975 26.67 0)
+			(at 336.8675 21.59 0)
 			(effects
 				(font
@@
 		)
 		(property "Footprint" "Diode_SMD:Nexperia_CFP3_SOD-123W"
-			(at 335.28 26.035 0)
+			(at 336.55 20.955 0)
 			(effects
 				(font
@@
 		)
 		(property "Datasheet" "https://assets.nexperia.com/documents/data-sheet/PMEG6020ER.pdf"
-			(at 335.28 30.48 0)
+			(at 336.55 25.4 0)
 			(effects
 				(font
@@
 		)
 		(property "Description" "60V, 2A low Vf MEGA Schottky barrier rectifier, SOD-123W"
-			(at 335.28 30.48 0)
+			(at 336.55 25.4 0)
 			(effects
 				(font
